File: leistungsstromquelle.kicad_pcb (KiCad board)
At the start: 2 copper layers, 71 parts, among them J1 OSTTC022162, J2 640456-2, J3 OSTTC022162, J4 640456-3, J5 640456-3, J6 640456-2, K1 FRT5_separated, Q1 BS250, Q2 2N7000, Q3 2N7000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

Commit message: minor changes
Parts:
- added G***: LOGO, kicad_logos:cerasus_loogo_klein, F.Cu at (262.9, 139.7)
- added G***: LOGO, kicad_logos:cherry_logo_2, F.Cu at (261.6, 141.0)
