File: leistungsstromquelle.sch (KiCad schematic (older format))
At the start: 71 parts, among them J1 OSTTC022162, J2 Conn_01x02_Male, J3 OSTTC022162, J4 Conn_01x03_Male, J7 Conn_01x03_Male, K1 FRT5_separated, Q1 BS250, Q2 2N7000, Q3 2N7000, Q4 TIP142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

Commit message: structured
Parts:
- removed C1, C14, C15, C4, C8, C9: 1u, Capacitor_THT:CP_Radial_D5.0mm_P2.50mm, symbol Device:CP
- removed C11, C2, C5: 10n, Capacitor_THT:C_Disc_D10.0mm_W2.5mm_P5.00mm, symbol Device:C
- removed C12, C3, C6: 100p, Capacitor_THT:C_Disc_D10.0mm_W2.5mm_P5.00mm, symbol Device:C
- removed C17: 10n, Capacitor_THT:C_Disc_D10.5mm_W5.0mm_P10.00mm, symbol Device:C
- removed C18: 100p, Capacitor_THT:C_Disc_D10.5mm_W5.0mm_P10.00mm, symbol Device:C
- removed D1: LED, LED_THT:LED_D5.0mm, symbol Device:LED
- removed D2: 1N4001, Diode_THT:D_DO-41_SOD81_P10.16mm_Horizontal, symbol Diode:1N4001
- removed F1: Fuse, Fuse:Fuseholder_Cylinder-5x20mm_EATON_HBW_Vertical_Closed, symbol Device:Fuse
- removed J1: OSTTC022162, digikey-footprints:Term_Block_1x2_P5.08MM, symbol dk_Terminal-Blocks-Wire-to-Board:OSTTC022162
- removed J?: Conn_01x02_Male, symbol Connector:Conn_01x02_Male
- removed unit 1 of K1
- removed unit 2 of K1
- removed R17: 2k3, Resistor_THT:R_Axial_DIN0207_L6.3mm_D2.5mm_P7.62mm_Horizontal, symbol Device:R
- removed R18, R19: 240, Resistor_THT:R_Axial_DIN0207_L6.3mm_D2.5mm_P7.62mm_Horizontal, symbol Device:R
- removed RV3: 2k, Potentiometer_THT:Potentiometer_Bourns_3296W_Vertical, symbol Device:R_POT_TRIM
- removed unit 3 of U1
- removed unit 5 of U2
- removed U3: LM317T, digikey-footprints:TO-220-3, symbol dk_PMIC-Voltage-Regulators-Linear:LM317T
- removed U4: LM317L_TO92, Package_TO_SOT_THT:TO-92_Inline, symbol Regulator_Linear:LM317L_TO92
- added C3, C6: 1u, Capacitor_THT:CP_Radial_D5.0mm_P2.50mm, symbol Device:CP
- added D1: 1N4001, Diode_THT:D_DO-41_SOD81_P10.16mm_Horizontal, symbol Diode:1N4001
- added D2: LED, LED_THT:LED_D5.0mm, symbol Device:LED
- added K2: FRT5_separated, Relay_THT:Relay_DPDT_FRT5, symbol Relay:FRT5_separated
- added U5: LM393, digikey-footprints:DIP-8_W7.62mm, symbol Comparator:LM393
- added U6: TL074, Package_DIP:DIP-14_W7.62mm_Socket, symbol Amplifier_Operational:TL074
- C13: value 100p -> 10n
- C16: value 10n -> 100p; footprint Capacitor_THT:C_Disc_D10.5mm_W5.0mm_P10.00mm -> Capacitor_THT:C_Disc_D10.0mm_W2.5mm_P5.00mm
- C19: footprint Capacitor_THT:C_Disc_D10.5mm_W5.0mm_P10.00mm -> Capacitor_THT:C_Disc_D10.0mm_W2.5mm_P5.00mm
- R1: value 10k -> 0
- R2: value 10k -> 1k5
- R4: value 1Meg -> 10k
- R5: value 1k5 -> 10k
- R6: value 0 -> 1Meg
Connections:
- net +12V: now also C13.1, C19.1, R2.1, R3.1, C6.1, U5.8 (V+); no longer C16.1, R1.1, R5.1
- net GND: now also R4.2, C3.2, C6.2, D2.1 (K), U5.4 (V-), U6.11 (V-); no longer D3.1 (K), R2.2
- net VCC: now also C16.1, C3.1, U6.4 (V+); no longer C13.1
- net overtemp: now also D4.1 (K), R6.1; no longer R4.1
- net at R5.2: now also U2.1, U2.2 (-)
- net at Q2.3 (D): now also D3.1 (K); no longer D4.1 (K)
- net at SW2.1: now also D1.1 (K), K2.1, K2.3
- net at SW1.1 (A), SW2.2: now also K2.4
- net at D3.2 (A): now also R2.2; no longer R6.2
- net +5V renamed Stromversorgung/soll_max
- net Stromversorgung/soll_max: no longer C19.1
- new net: D2.2 (A), R1.2
- new net: D1.2 (A), K2.10, R1.1
- new net: R3.2, R4.1, U2.5 (+)
- new net: R5.1, R6.2, U1.3 (+)
Other:
- note added: "Ein- / Aus- / Temperaturabschaltung \nund Übertemperaturanzeige"
- note added: "Versorgung Komparator"
- note added: "Versorgung Operationsverstärker"
- note removed: "Anschluß Versorgungsspannung \nbzw. Eingang der Stromsenke"
- note removed: "Ein- / Aus- / Temperaturabschaltung und Übertemperaturanzeige"
- note removed: "VCC: 15V … 30V\nabs. max. 35V"
- note removed: "Versorgung 12 V"
- note removed: "Versorgung Komparator und Operationsverstärker"
- note removed: "Versorgung Lüfter"
- note removed: "max. Strom-Sollwert 5A -> 5V\nModifikation über RV3"
- moved on the sheet: C7, J2, J3, J4, J7, K1C, Q3, Q4, Q5, Q6, Q7, Q8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
