File: file5FCFCB3A.sch (KiCad schematic (older format))
At the start: 53 parts, among them J5 Conn_01x02_Male, J6 Conn_01x03_Male, J7 Conn_01x02_Male, Q3 BC857, Q4 BC857, Q5 BC860, Q6 BC850, Q7 BD139, Q8 BC847, Q9 BC847, U1 OP275, U2 LM317_TO-220

Commit message: pcb netzteil rev. 1.0 finished
Parts:
- removed C10, C?: 10u, Capacitor_SMD:C_1206_3216Metric_Pad1.42x1.75mm_HandSolder, symbol Device:C
- removed C5, C?: 1n, Capacitor_SMD:C_1206_3216Metric_Pad1.42x1.75mm_HandSolder, symbol Device:C
- removed C7, C?: 100n, Capacitor_SMD:C_1206_3216Metric_Pad1.42x1.75mm_HandSolder, symbol Device:C
- removed Q3, Q4: BC857, Package_TO_SOT_SMD:SOT-23, symbol Transistor_BJT:BC857
- removed R3: 4k7, Resistor_SMD:R_1206_3216Metric_Pad1.42x1.75mm_HandSolder, symbol Device:R
- removed R4: 220, Resistor_SMD:R_1206_3216Metric_Pad1.42x1.75mm_HandSolder, symbol Device:R
- removed U1: OP275, Package_SO:SOIC-8-1EP_3.9x4.9mm_P1.27mm_EP2.95x4.9mm_Mask2.71x3.4mm, symbol Amplifier_Operational:OP275
- removed Z1: 1N5222B, digikey-footprints:DO-35, symbol dk_Diodes-Zener-Single:1N5231BTR
- added C1, C11, C12: 1u, Capacitor_SMD:C_1206_3216Metric_Pad1.42x1.75mm_HandSolder, symbol Device:C
- added C6, C8, C9: 10n, Capacitor_SMD:C_1206_3216Metric_Pad1.42x1.75mm_HandSolder, symbol Device:C
- added R11, R8: 10k, Resistor_SMD:R_1206_3216Metric_Pad1.42x1.75mm_HandSolder, symbol Device:R
- added R9: 5k, Resistor_SMD:R_1206_3216Metric_Pad1.42x1.75mm_HandSolder, symbol Device:R
- added TP4, TP6: TestPoint, TestPoint:TestPoint_Loop_D2.50mm_Drill1.0mm, symbol Connector:TestPoint
- added U1: ADR421ARMZ, Package_SO:MSOP-8_3x3mm_P0.65mm, symbol Reference_Voltage:ADR421ARMZ
- added U2: OP07, Package_SO:SOIC-8_3.9x4.9mm_P1.27mm, symbol Amplifier_Operational:OP07
- C13: value 3300u -> 1500u; footprint Capacitor_THT:CP_Radial_D16.0mm_P7.50mm -> Capacitor_THT:CP_Radial_D12.5mm_P5.00mm
- C14: value 33u -> 15u
- C15: value 330n -> 150n
- C2: value 220n -> 100n
- D4: renamed from D5; footprint LED_SMD:LED_0805_2012Metric_Pad1.15x1.40mm_HandSolder -> LED_SMD:LED_1206_3216Metric_Pad1.42x1.75mm_HandSolder
- R1: renamed from R5; value 10k -> 7k4
- R2, R3: renamed from R?; value 1 -> 1R2
- R5: renamed from R9; value 18k -> 15k
- TP1, TP2, TP3: footprint TestPoint:TestPoint_Pad_D2.0mm -> TestPoint:TestPoint_Loop_D2.50mm_Drill1.0mm
- TP5: renamed from TP4; footprint TestPoint:TestPoint_Pad_D2.0mm -> TestPoint:TestPoint_Loop_D2.50mm_Drill1.0mm
- TP7: renamed from TP5; footprint TestPoint:TestPoint_Pad_D2.0mm -> TestPoint:TestPoint_Loop_D2.50mm_Drill1.0mm
- TP8: renamed from TP6; footprint TestPoint:TestPoint_Pad_D2.0mm -> TestPoint:TestPoint_Loop_D2.50mm_Drill1.0mm
- gave numbers to parts that had none: 1
- renumbered C12 to C10, C1 to C3, C3 to C4, C4 to C5, C9 to C7, D2 to D1, D3 to D2, D4 to D3, Q5 to Q1, Q6 to Q2, Q7 to Q3, Q8 to Q4, Q9 to Q5, R12 to R10, R13 to R12, R14 to R13, R15 to R14, R16 to R15, R8 to R4, R10 to R6, U2 to U3
Connections:
- net -2V5: now also C6.1, R11.1, TP6.1, U2.6; no longer C2.1
- net at D4.1 (K), J7.1 (Pin_1): no longer Q5.3 (C)
- net +12V_in renamed V+
- net V+: now also C2.1, C1.1, C11.1, C8.1, U1.2 (VIN), U2.7 (V+)
- net GND_in renamed GND
- net GND: now also C1.2, C11.2, C12.1, C6.2, C8.2, C9.1, R9.1, U1.4 (GND)
- net Ua_out renamed Ua_aus
- net Ua_aus: no longer J7.2 (Pin_2)
- new net: R8.2, TP4.1, U1.6 (OUT)
- new net: R11.2, R8.1, U2.2 (-)
- new net: R9.2, U2.3 (+)
- new net: J7.2 (Pin_2), Q5.3 (C)
- new net V-: C12.2, C9.2, U2.4 (V-)
- no-connect marks 1 -> 3
Other:
- note added: "Spannungsreferenz -2.5V:"
- note added: "einstellbare (0V … ca. 13V) \nund strombegrenzte (I_max = 0,65V / 0,6Ohm = 1.1A)\ngeregelte Spannung:"
- note removed: "Erzeugung neg. Referenzspannung von -2.5V: \nKonstantstromquelle treibt konstanten Strom durch \nZ-Diode und Spannungsabfall wird von OP invertiert"
- note removed: "I_Z_const ca. \n0.65V/220Ohm \n= 3mA"
- note removed: "OpAmp OP275\nmit maximal\n+/- 23mA\nbelasten!"
- note removed: "einstellbare (0V … ca. 10V) \nund strombegrenzte (I_max=1A)\ngeregelte Spannung"
- moved on the sheet: C10, C3, C4, C5, C7, D1, D2, D3, D4, HS1, J5, J6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
