File: netzteil.sch (KiCad schematic (older format))
At the start: 78 parts, among them J1 OSTTC022162, J2 OSTTC022162, J3 Conn_01x02_Male, J4 Conn_01x02_Male, J5 Conn_01x02_Male, J6 Conn_01x02_Male, J7 Conn_01x02_Male, J8 Conn_01x02_Male, J9 Conn_01x02_Male, Q1 SUD50P10-43L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

Commit message: change to SMD 1206 and restructuring
Parts:
- removed C1, C20: 100u, Capacitor_THT:CP_Radial_D5.0mm_P2.50mm, symbol Device:CP
- removed C10, C21, C23, C8: 4700u, symbol Device:CP
- removed C12: 22p, Capacitor_THT:C_Disc_D10.5mm_W5.0mm_P10.00mm, symbol Device:C
- removed C13, C19, C31: 100n, Capacitor_THT:C_Disc_D10.5mm_W5.0mm_P10.00mm, symbol Device:C
- removed C15, C17, C26, C28: 470n, Capacitor_THT:C_Disc_D10.5mm_W5.0mm_P10.00mm, symbol Device:C
- removed C16, C29, C3, C7: 1000u, Capacitor_THT:CP_Radial_D5.0mm_P2.50mm, symbol Device:CP
- removed C18, C30, C9: 10u, Capacitor_THT:C_Disc_D10.5mm_W5.0mm_P10.00mm, symbol Device:C
- removed C2, C22: 1u, Capacitor_THT:C_Disc_D10.0mm_W2.5mm_P5.00mm, symbol Device:C
- removed C27, C4: 10n, Capacitor_THT:C_Disc_D10.0mm_W2.5mm_P5.00mm, symbol Device:C
- removed C5: 10u, Capacitor_THT:C_Disc_D10.0mm_W2.5mm_P5.00mm, symbol Device:C
- removed C6, C?: 100n, Capacitor_THT:C_Disc_D10.0mm_W2.5mm_P5.00mm, symbol Device:C
- removed C? (x2): 10u, Capacitor_THT:CP_Radial_D5.0mm_P2.50mm, symbol Device:CP
- removed C? (x4): 47u, symbol Device:CP
- removed D1, D4, D? (x2): 1N4002, Diode_THT:D_DO-41_SOD81_P10.16mm_Horizontal, symbol Diode:1N4002
- removed D2: BZX84Cxx, Diode_SMD:D_SOT-23_ANK, symbol Diode:BZX84Cxx
- removed D3: 1.5KExxCA, Diode_THT:D_DO-201AE_P15.24mm_Horizontal, symbol Diode:1.5KExxCA
- removed F2: Fuse, Fuse:Fuseholder_Cylinder-5x20mm_EATON_HBW_Vertical_Closed, symbol Device:Fuse
- removed FL1, FL2: EMI_Filter_LL_1423, symbol Device:EMI_Filter_LL_1423
- removed HS1, HS2, HS3: Heatsink, Heatsink:Heatsink_Fischer_SK129-STS_42x25mm_2xDrill2.5mm, symbol Mechanical:Heatsink
- removed J2: OSTTC022162, digikey-footprints:Term_Block_1x2_P5.08MM, symbol dk_Terminal-Blocks-Wire-to-Board:OSTTC022162
- removed J3, J6, J7, J8, J9: Conn_01x02_Male, Connector_PinHeader_2.54mm:PinHeader_1x02_P2.54mm_Vertical, symbol Connector:Conn_01x02_Male
- removed J5: Conn_01x02_Male, symbol Connector:Conn_01x02_Male
- removed PS1: IRM-60-24, CONV_IRM-60-48, symbol IRM-60-24:IRM-60-24
- removed Q1: SUD50P10-43L, Package_TO_SOT_SMD:TO-252-2, symbol Transistor_FET:SUD50P10-43L
- removed Q2: TIP122, Package_TO_SOT_THT:TO-220-3_Vertical, symbol Transistor_BJT:TIP122
- removed R3: 1k, Resistor_THT:R_Axial_DIN0207_L6.3mm_D2.5mm_P10.16mm_Horizontal, symbol Device:R
- removed R4: 330, Resistor_THT:R_Axial_DIN0207_L6.3mm_D2.5mm_P10.16mm_Horizontal, symbol Device:R
- removed R5: 3k3, Resistor_THT:R_Axial_DIN0207_L6.3mm_D2.5mm_P10.16mm_Horizontal, symbol Device:R
- removed R6: 390, Resistor_THT:R_Axial_DIN0207_L6.3mm_D2.5mm_P10.16mm_Horizontal, symbol Device:R
- removed RV1: 100k, symbol Device:R_POT
- removed TP1, TP2, TP3, TP4, TP5: TestPoint, symbol Connector:TestPoint
- removed U1, U3: LM317T, digikey-footprints:TO-220-3, symbol dk_PMIC-Voltage-Regulators-Linear:LM317T
- removed U2: TL072, symbol Amplifier_Operational:TL072
- added D1: LED, LED_SMD:LED_0805_2012Metric_Pad1.15x1.40mm_HandSolder, symbol Device:LED
- added J2: Conn_01x02_Male, Connector_PinHeader_2.54mm:PinHeader_1x02_P2.54mm_Vertical, symbol Connector:Conn_01x02_Male
- added J3: Conn_01x03_Male, Connector_PinHeader_2.54mm:PinHeader_1x03_P2.54mm_Vertical, symbol Connector:Conn_01x03_Male
- added Q1, Q2: BC847, Package_TO_SOT_SMD:SOT-23, symbol Transistor_BJT:BC847
- H1, H2, H3, H4: footprint MountingHole:MountingHole_2.7mm -> MountingHole:MountingHole_3.2mm_M3_DIN965
- J4: footprint (none) -> Connector_PinHeader_2.54mm:PinHeader_1x02_P2.54mm_Vertical
- R1: value 100k -> 4k7; footprint (none) -> Resistor_SMD:R_1206_3216Metric_Pad1.42x1.75mm_HandSolder
- R2: value 50k -> 100; footprint (none) -> Resistor_SMD:R_1206_3216Metric_Pad1.42x1.75mm_HandSolder
Connections:
- net labels added: -12V, GND1, Ua
- net labels removed: +24V, +5V
- wire segments 266 -> 53
Other:
- note added: "Anzeige: \nSpannungsversorgung\nvorhanden"
- note added: "Versorgung +12V/-12V"
- note added: "min. 28VDC bis \nmax. 37.4VDC"
- note removed: "Anschluß Versorgungsspannung \nbzw. Eingang der Stromsenke"
- note removed: "Einstellbare Spannung\n0V … ca. 20V"
- note removed: "Umschalter:\n1 -> 1: Stromquelle mit VCC = 24V\n2 -> 1: Stromsenke / elektr. Last"
- note removed: "VCC: 15V … 30V\nabs. max. 35V"
- note removed: "Verpolschutz"
- note removed: "Versorgung 12 V"
- note removed: "Versorgung 12V"
- note removed: "Versorgung 24V"
- note removed: "Versorgung 5 V"
- note removed: "Versorgung 5V"
- note removed: "Versorgung VCC"
- moved on the sheet: H1

Commit message: pcb netzteil rev. 1.0 finished
Parts:
- removed D1: LED, LED_SMD:LED_0805_2012Metric_Pad1.15x1.40mm_HandSolder, symbol Device:LED
- removed F1: Fuse, Fuse:Fuseholder_Cylinder-5x20mm_EATON_HBW_Vertical_Closed, symbol Device:Fuse
- removed J1: OSTTC022162, digikey-footprints:Term_Block_1x2_P5.08MM, symbol dk_Terminal-Blocks-Wire-to-Board:OSTTC022162
- removed J2, J4: Conn_01x02_Male, Connector_PinHeader_2.54mm:PinHeader_1x02_P2.54mm_Vertical, symbol Connector:Conn_01x02_Male
- removed J3: Conn_01x03_Male, Connector_PinHeader_2.54mm:PinHeader_1x03_P2.54mm_Vertical, symbol Connector:Conn_01x03_Male
- removed Q1, Q2: BC847, Package_TO_SOT_SMD:SOT-23, symbol Transistor_BJT:BC847
- removed R1: 4k7, Resistor_SMD:R_1206_3216Metric_Pad1.42x1.75mm_HandSolder, symbol Device:R
- removed R2: 100, Resistor_SMD:R_1206_3216Metric_Pad1.42x1.75mm_HandSolder, symbol Device:R
- added J1: Screw_Terminal_01x04, TerminalBlock_Phoenix:TerminalBlock_Phoenix_MKDS-3-4-5.08_1x04_P5.08mm_Horizontal, symbol Connector:Screw_Terminal_01x04
- added J2, J3: Screw_Terminal_01x03, TerminalBlock:TerminalBlock_bornier-3_P5.08mm, symbol Connector:Screw_Terminal_01x03
Connections:
- net GND: now also J2.2 (Pin_2), J3.2 (Pin_2)
- new net 15V/-15V gesiebt/+15V_aus: J3.1 (Pin_1)
- new net 15V/-15V gesiebt/-15V_aus: J3.3 (Pin_3)
- new net 15V/-15V gesiebt/VDC+: J2.1 (Pin_1)
- new net 15V/-15V gesiebt/VDC-: J2.3 (Pin_3)
- new net Verpolschutz und Filterung/V+1: J1.4 (Pin_4)
- new net Verpolschutz und Filterung/V+2: J1.2 (Pin_2)
- new net Verpolschutz und Filterung/V-1: J1.3 (Pin_3)
- new net Verpolschutz und Filterung/V-2: J1.1 (Pin_1)
Other:
- note added: "Versorgung +15V/-15V"
- note added: "Versorgung +VDC/-VDC"
- note removed: "Anzeige: \nSpannungsversorgung\nvorhanden"
- note removed: "Versorgung +12V/-12V"
- note removed: "min. 28VDC bis \nmax. 37.4VDC"
- moved on the sheet: H1, H2, H3, H4
