File: steuerung_ueberwachung_analog.sch (KiCad schematic (older format))
At the start: 55 parts, among them J10 Conn_01x02_Male, J11 Conn_01x03_Male, J12 Conn_01x02_Male, J13 Conn_01x01_Male, J14 Conn_01x03_Male, J15 Conn_01x02_Male, J16 Conn_01x02_Male, Q3 2N7000, Q4 2N7000, Q5 2N7000, SW1 SW_Push, SW2 SW_Push, U4 NE555P, U5 TL074, U6 LM393

Commit message: change to SMD 1206 and restructuring
Parts:
- removed C36: 47n, symbol Device:C
- removed J13: Conn_01x01_Male, symbol Connector:Conn_01x01_Male
- added J10: Conn_01x03_Male, symbol Connector:Conn_01x03_Male
- added J14: Conn_01x02_Male, symbol Connector:Conn_01x02_Male
- 100k1: renamed from R11; value 100 -> 100k
- C39: renamed from C?; value 4u7 -> 100n
- R36: renamed from R22; value 10k -> 18k
- R37: renamed from R23; value 10k -> 18k
- U5: renamed from U4; footprint Package_DIP:DIP-8_W7.62mm -> Package_DIP:DIP-8_W7.62mm_Socket
- U6: renamed from U5; footprint (none) -> Package_DIP:DIP-8_W7.62mm_Socket
- U7: renamed from U6; footprint (none) -> Package_DIP:DIP-8_W7.62mm_Socket
- U7: renamed from U6; footprint digikey-footprints:DIP-8_W7.62mm -> Package_DIP:DIP-8_W7.62mm_Socket
- renumbered C37 to C40, C38 to C41, C39 to C42, C40 to C43, C41 to C44, C42 to C45, C43 to C46, C44 to C47, D5 to D15, D6 to D16, J12 to J11, J14 to J12, J15 to J13, J16 to J15, J10 to J8, J11 to J9, Q3 to Q12, Q4 to Q13, Q5 to Q14, R7 to R22, R8 to R23, R9 to R24, R10 to R25, R12 to R26, R13 to R27, R14 to R28, R15 to R29, R16 to R30, R17 to R31, R18 to R32, R19 to R33, R20 to R34, R21 to R35, RV2 to RV3, RV3 to RV4, TP6 to TP12, TP7 to TP13, TP8 to TP14, TP9 to TP15, TP10 to TP16, TP11 to TP17, TP12 to TP18, TP13 to TP19, TP14 to TP20
Connections:
- net labels added: -12V
- wire segments 171 -> 176
Other:
- note added: "Versorgung +12V/-12V"
- note added: "maximaler Sollwert \n(100mV -> 1A)"
- note removed: "f_g ca. 2.13 kHz"
- note removed: "maximaler Sollwert (100mV -> 1A)"
- moved on the sheet: 100k1, C39, J11, TP12

Commit message: pcb netzteil rev. 1.0 finished
Changed lines of the file:
@@
 $Descr A4 11693 8268
 encoding utf-8
-Sheet 5 8
+Sheet 1 3
 Title "Leistungsstromquelle/-senke"
 Date "01.06.2020"
@@
 	2850 4150 2900 4150
 $Sheet
-S 4650 3500 950  700
+S 4650 2200 950  700
 U 60068EBE
 F0 "Versorgungen & Mechanik" 50
@@
 	0    1    1    0
 $EndComp
+$Sheet
+S 4750 3450 1200 850
+U 5F28C6A8
+F0 "Sollwert" 50
+F1 "file5F28C6A7.sch" 50
+$EndSheet
 $EndSCHEMATC
