File: file60AF546E.sch (KiCad schematic (older format))
At the start: 31 parts, among them U3 LM317_TO-220, U4 LM337_TO220

Commit message: pcb netzteil rev. 1.0 finished
Parts:
- removed C25, C26: 3300u, Capacitor_THT:CP_Radial_D16.0mm_P7.50mm, symbol Device:CP
- removed C27, C?: 33u, Capacitor_SMD:C_1206_3216Metric_Pad1.42x1.75mm_HandSolder, symbol Device:C
- removed C33, C34: 330u, Capacitor_THT:CP_Radial_D10.0mm_P5.00mm, symbol Device:CP
- removed C35, C?: 3u3, Capacitor_SMD:C_1206_3216Metric_Pad1.42x1.75mm_HandSolder, symbol Device:C
- removed C37, C?: 33n, Capacitor_SMD:C_1206_3216Metric_Pad1.42x1.75mm_HandSolder, symbol Device:C
- removed C?: 330n, Capacitor_SMD:C_1206_3216Metric_Pad1.42x1.75mm_HandSolder, symbol Device:C
- removed D11, D12: 1N4002, Diode_THT:D_DO-41_SOD81_P10.16mm_Horizontal, symbol Diode:1N4002
- added C13, C14: 470u, Capacitor_THT:CP_Radial_D12.5mm_P5.00mm, symbol Device:CP
- added C15, C16: 4u7, Capacitor_SMD:C_1206_3216Metric_Pad1.42x1.75mm_HandSolder, symbol Device:C
- added C17, C18: 47n, Capacitor_SMD:C_1206_3216Metric_Pad1.42x1.75mm_HandSolder, symbol Device:C
- added C19, C20: 330u, Capacitor_THT:CP_Radial_D10.0mm_P5.00mm, symbol Device:CP
- added C21, C22: 3u3, Capacitor_SMD:C_1206_3216Metric_Pad1.42x1.75mm_HandSolder, symbol Device:C
- added C23, C24: 33n, Capacitor_SMD:C_1206_3216Metric_Pad1.42x1.75mm_HandSolder, symbol Device:C
- added C27, C28: 1500u, Capacitor_THT:CP_Radial_D12.5mm_P5.00mm, symbol Device:CP
- added C30: 15u, Capacitor_SMD:C_1206_3216Metric_Pad1.42x1.75mm_HandSolder, symbol Device:C
- added C31, C32: 150n, Capacitor_SMD:C_1206_3216Metric_Pad1.42x1.75mm_HandSolder, symbol Device:C
- added D10, D9: MRA4003T3G, Diode_SMD:D_SMA, symbol Diode:MRA4003T3G
- added HS1, HS2: Heatsink, Heatsink:Heatsink_Fischer_SK104-STC-STIC_35x13mm_2xDrill2.5mm, symbol Mechanical:Heatsink
- added Q7: TIP120, Package_TO_SOT_THT:TO-220-3_Vertical, symbol Transistor_BJT:TIP120
- added Q8: TIP125, Package_TO_SOT_THT:TO-220-3_Vertical, symbol Transistor_BJT:TIP125
- added R10, R9: 220, Resistor_SMD:R_1206_3216Metric_Pad1.42x1.75mm_HandSolder, symbol Device:R
- added R11, R12: 1Meg, Resistor_SMD:R_1206_3216Metric_Pad1.42x1.75mm_HandSolder, symbol Device:R
- added TP10, TP11: TestPoint, TestPoint:TestPoint_Loop_D2.50mm_Drill1.0mm, symbol Connector:TestPoint
- C29: value 330n -> 15u
- RV1, RV2: value 2k -> 5k
- TP12: renamed from TP9; footprint TestPoint:TestPoint_Pad_D2.0mm -> TestPoint:TestPoint_Loop_D2.50mm_Drill1.0mm
- TP13: renamed from TP10; footprint TestPoint:TestPoint_Pad_D2.0mm -> TestPoint:TestPoint_Loop_D2.50mm_Drill1.0mm
- TP14: renamed from TP11; footprint TestPoint:TestPoint_Pad_D2.0mm -> TestPoint:TestPoint_Loop_D2.50mm_Drill1.0mm
- renumbered C31 to C25, C32 to C26, D13 to D11, D14 to D12, D9 to D7, D10 to D8, R20 to R13, R21 to R14, U3 to U1, U4 to U2
Connections:
- net at C25.1, R13.2, RV1.3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: now also D9.2 (A)
- net at C26.2, R14.1, RV2.3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: now also D10.1 (K)
- net +12V_out renamed +15V_aus
- net +15V_aus: now also C29.1, C27.1, C31.1, D9.1 (K)
- net -12V_out renamed -15V_aus
- net -15V_aus: now also C28.2, C30.2, C32.2, D10.2 (A)
- net GND_ein: no longer names the net of D8.2 (A), U2.2 (VI)
- net GND_ein: now also C20.2, C22.2, C24.2, Q8.3 (E), TP11.1
- net GND_out renamed GND_aus
- net GND_aus: now also C13.2, C14.1, C15.2, C16.1, C17.2, C18.1, C19.2, C20.1, C21.2, C22.1, C23.2, C24.1, C27.2, C28.1, C30.1, C31.2, C32.1, R11.2, R12.1
- net VCC_ein: no longer names the net of D7.1 (K), U1.3 (VI)
- net VCC_ein: now also C19.1, C21.1, C23.1, Q7.3 (E), TP10.1; no longer C29.1
- new net: C13.1, C15.1, C17.1, Q7.1 (B), R11.1, R9.1
- new net: C14.2, C16.2, C18.2, Q8.1 (B), R10.1, R12.2
- new net VDC+: Q7.2 (C), R9.2
- new net VDC-: Q8.2 (C), R10.2
Other:
- note added: "+15V/-15V -> RV1 = RV2 = 2640 Ohm"
- note added: "fg=1.5Hz"
- moved on the sheet: C25, C26, D11, D12, D7, D8, HS3, HS4, R13, R14, RV1, RV2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

Commit message: photo added
Parts:
- C19, C20: value 330u -> 100u
- C25, C26: footprint Capacitor_SMD:C_0805_2012Metric_Pad1.15x1.40mm_HandSolder -> Capacitor_SMD:C_1206_3216Metric_Pad1.42x1.75mm_HandSolder
Changed lines of the file:
@@
 F 0 "C25" H 5665 3596 50  0000 L CNN
 F 1 "10u" H 5665 3505 50  0000 L CNN
-F 2 "Capacitor_SMD:C_0805_2012Metric_Pad1.15x1.40mm_HandSolder" H 5588 3400 50  0001 C CNN
+F 2 "Capacitor_SMD:C_1206_3216Metric_Pad1.42x1.75mm_HandSolder" H 5588 3400 50  0001 C CNN
 F 3 "~" H 5550 3550 50  0001 C CNN
 	1    5550 3550
@@
 F 0 "C26" H 5665 3996 50  0000 L CNN
 F 1 "10u" H 5665 3905 50  0000 L CNN
-F 2 "Capacitor_SMD:C_0805_2012Metric_Pad1.15x1.40mm_HandSolder" H 5588 3800 50  0001 C CNN
+F 2 "Capacitor_SMD:C_1206_3216Metric_Pad1.42x1.75mm_HandSolder" H 5588 3800 50  0001 C CNN
 F 3 "~" H 5550 3950 50  0001 C CNN
 	1    5550 3950
@@
 AR Path="/60AF546F/5F1D8CF0" Ref="C19"  Part="1"
 F 0 "C19" H 4050 3500 50  0000 L CNN
-F 1 "330u" V 4200 3250 50  0000 L CNN
+F 1 "100u" V 4200 3250 50  0000 L CNN
 F 2 "Capacitor_THT:CP_Radial_D10.0mm_P5.00mm" H 4088 3250 50  0001 C CNN
 F 3 "~" H 4050 3400 50  0001 C CNN
@@
 AR Path="/60AF546F/5F1DEC53" Ref="C20"  Part="1"
 F 0 "C20" H 4050 4250 50  0000 L CNN
-F 1 "330u" V 4200 4000 50  0000 L CNN
+F 1 "100u" V 4200 4000 50  0000 L CNN
 F 2 "Capacitor_THT:CP_Radial_D10.0mm_P5.00mm" H 4088 4000 50  0001 C CNN
 F 3 "~" H 4050 4150 50  0001 C CNN
